Commit message: fixed camera height

File: ME461LABS_ws/src/sokoban/urdf/camera.xacro (robot description, xacro)
@@ -23,5 +23,5 @@
         <parent link="world" />
         <child link="camera_link" />
-        <origin xyz="0 0 20.0" rpy="0 ${pi / 2.0} 0" />
+        <origin xyz="0 0 10.0" rpy="0 ${pi / 2.0} 0" />
     </joint>
     <link name="camera_link_optical">
