Commit message: Added launch file for spawning targets, fixed the appearance of targets

File: ME461LABS_ws/src/sokoban/urdf/box_gazebo.xacro (robot description, xacro)
@@ -2,5 +2,5 @@
 <robot xmlns:xacro="http://www.ros.org/wiki/xacro">
     <gazebo reference = "box_link">
-        <material>Gazebo/Red</material>
+        <material>Gazebo/Yellow</material>
     </gazebo>
 </robot>

File: ME461LABS_ws/src/sokoban/urdf/camera.xacro (robot description, xacro)
@@ -23,5 +23,5 @@
         <parent link="world" />
         <child link="camera_link" />
-        <origin xyz="0 0 10.0" rpy="0 ${pi / 2.0} 0" />
+        <origin xyz="0 0 25.0" rpy="0 ${pi / 2.0} 0" />
     </joint>
     <link name="camera_link_optical">
@@ -36,5 +36,5 @@
     </joint>
     <gazebo reference="camera_link">
-        <material>Gazebo/Red</material>
+        <material>Gazebo/DarkGrey</material>
         <sensor name="camera_sensor" type="camera">
             <pose>0 0 0 0 0 0</pose>
