Commit message: Added the turtlebot3

File: ME461LABS_ws/src/sokoban/urdf/box.xacro (robot description, xacro)
@@ -1,7 +1,7 @@
 <?xml version="1.0"?>
 <robot xmlns:xacro="http://www.ros.org/wiki/xacro">
-    <xacro:property name="base_length" value="1.0" />
-    <xacro:property name="base_width" value="1.0" />
-    <xacro:property name="base_height" value="1.0" />
+    <xacro:property name="base_length" value="0.5" />
+    <xacro:property name="base_width" value="0.5" />
+    <xacro:property name="base_height" value="0.5" />
     <link name="world"></link>
     <link name="box_link">

Commit message: Enhanced the outlook of turtlebot3

File: ME461LABS_ws/src/sokoban/urdf/box.xacro (robot description, xacro)
@@ -1,7 +1,7 @@
 <?xml version="1.0"?>
 <robot xmlns:xacro="http://www.ros.org/wiki/xacro">
-    <xacro:property name="base_length" value="0.5" />
-    <xacro:property name="base_width" value="0.5" />
-    <xacro:property name="base_height" value="0.5" />
+    <xacro:property name="base_length" value="0.2" />
+    <xacro:property name="base_width" value="0.2" />
+    <xacro:property name="base_height" value="0.2" />
     <link name="world"></link>
     <link name="box_link">
@@ -19,5 +19,5 @@
             <origin xyz="0 0 ${base_height / 2.0}" rpy="0 0 0" />
         </collision>
-        <xacro:box_inertia m="5.0" l="${base_length}" w="${base_width}" h="${base_height}"
+        <xacro:box_inertia m="0.1" l="${base_length}" w="${base_width}" h="${base_height}"
                            xyz="0 0 ${base_height / 2.0}" rpy="0 0 0" />
     </link>

Commit message: size adjusted, direction pointer added

File: ME461LABS_ws/src/sokoban/urdf/box.xacro (robot description, xacro)
@@ -1,7 +1,7 @@
 <?xml version="1.0"?>
 <robot xmlns:xacro="http://www.ros.org/wiki/xacro">
-    <xacro:property name="base_length" value="0.2" />
-    <xacro:property name="base_width" value="0.2" />
-    <xacro:property name="base_height" value="0.2" />
+    <xacro:property name="base_length" value="0.3" />
+    <xacro:property name="base_width" value="0.3" />
+    <xacro:property name="base_height" value="0.3" />
     <link name="world"></link>
     <link name="box_link">

File: ME461LABS_ws/src/sokoban/urdf/camera.xacro (robot description, xacro)
@@ -23,5 +23,5 @@
         <parent link="world" />
         <child link="camera_link" />
-        <origin xyz="0 0 25.0" rpy="0 ${pi / 2.0} 0" />
+        <origin xyz="0 0 6" rpy="0 ${pi / 2.0} 0" />
     </joint>
     <link name="camera_link_optical">
@@ -44,4 +44,10 @@
                 <frame_name>camera_link</frame_name>
             </plugin>
+            <camera>
+		<image>
+		  <width>1920</width>
+		  <height>1920</height>
+	        </image>
+	    </camera>
         </sensor>
     </gazebo>
